File: my-keeb.kicad_pcb (KiCad board)
At the start: 2 copper layers, 319.1 x 97.6 mm, 128 parts, among them SW1 SW_Push, SW10 SW_Push, SW11 SW_Push, SW12 SW_Push, SW13 SW_Push, SW14 SW_Push, SW15 SW_Push, SW16 SW_Push, SW17 SW_Push, SW18 SW_Push, SW19 SW_Push, SW2 SW_Push, SW20 SW_Push, SW21 SW_Push, SW22 SW_Push, SW23 SW_Push, SW24 SW_Push, SW25 SW_Push, SW26 SW_Push, SW27 SW_Push, SW28 SW_Push, SW29 SW_Push, SW3 SW_Push, SW30 SW_Push, SW31 SW_Push, SW32 SW_Push, SW33 SW_Push, SW34 SW_Push, SW35 SW_Push, SW36 SW_Push, SW37 SW_Push, SW38 SW_Push, SW39 SW_Push, SW4 SW_Push, SW40 SW_Push, SW41 SW_Push, SW42 SW_Push, SW43 SW_Push, SW44 SW_Push, SW45 SW_Push, SW46 SW_Push, SW47 SW_Push, SW48 SW_Push, SW49 SW_Push, SW5 SW_Push, SW50 SW_Push, SW51 SW_Push, SW52 SW_Push, SW53 SW_Push, SW54 SW_Push, SW55 SW_Push, SW56 SW_Push, SW57 SW_Push, SW58 SW_Push, SW59 SW_Push, SW6 SW_Push, SW60 SW_Push, SW61 SW_Push, SW7 SW_Push, SW8 SW_Push, SW9 SW_Push

Commit message: pcb fixes
Parts:
- moved A1 7.94 mm to (260.2, -136.3)
- moved D28 4.76 mm to (225.7, -95.2)
- moved D41 3.33 mm to (220.0, -76.2)
- moved D27 3.00 mm to (203.7, -95.2)
- moved D50 1.43 mm to (146.2, -57.1)
Routing:
- net /COL0: track 0.00 -> 392.0 mm
- net /COL1: track 0.00 -> 382.6 mm
- net /COL2: track 0.00 -> 363.2 mm
- net /ROW3: track 0.00 -> 338.7 mm
- net /ROW4: track 0.00 -> 334.2 mm
- net /ROW2: track 0.00 -> 328.3 mm
- net /ROW1: track 0.00 -> 322.3 mm
- net /COL3: track 0.00 -> 322.0 mm
- net /ROW0: track 0.00 -> 313.5 mm
- net /COL5: track 0.00 -> 310.3 mm
- net /COL4: track 0.00 -> 304.9 mm
- net /COL6: track 0.00 -> 273.1 mm
- net /COL8: track 0.00 -> 266.7 mm
- net /COL9: track 0.00 -> 256.4 mm
- net /COL7: track 0.00 -> 255.9 mm
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Other:
- board size 319.1 x 97.6 mm -> 319.1 x 102.4 mm

Commit message: gerber files and drill files with finishing pcb touches
Routing:
- added copper zone on B.Cu, net Net-(A1-GND-Pad13)
- added copper zone on F.Cu, net Net-(A1-GND-Pad13)
Changed lines of the file:
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@@
 		(net "Net-(D26-A)")
+	)
+	(zone
+		(net "Net-(A1-GND-Pad13)")
+		(layers "F.Cu" "B.Cu")
+		(name "ground")
+		(hatch edge 0.5)
+		(connect_pads
+			(clearance 0.5)
+		)
+		(min_thickness 0.25)
+		(fill yes
+			(thermal_gap 0.5)
+			(thermal_bridge_width 0.5)
+			(island_removal_mode 0)
+		)
+		(polygon
+			(pts
+				(xy -38.1 -138.1125) (xy -38.1 -35.71875) (xy 280.9875 -35.71875) (xy 280.9875 -138.1125)
+			)
+		)
 	)
 	(embedded_fonts no)

Commit message: pcb
Parts:
- added G***: LOGO, logos:manuul, F.Cu at (261.9, -47.6)
- D61: moved to B.Cu
- moved D61 7.62 mm to (244.3, -57.1), turned to 180 degrees
Routing:
- net /ROW4: track 334.2 -> 339.4 mm
- net Net-(D61-A): track 7.87 -> 5.10 mm
Other:
- board text added: "designed and assembled by tuguldur0"
